Commit message: add joint_states pub

File: diffdrive_description/urdf/diffdrive.urdf (robot description, URDF)
Before this commit: robot DiffDrive, 2 links, 4 joints
Joints:
- removed joint left_joint
- removed joint right_joint
- added joint left_wheel_joint: type continuous, parent base_link, child left_wheel_link, origin xyz=-0.1 0.1 -0.015 rpy=0.0 0.0 0.0, axis 0.0 1.0 0.0
- added joint right_wheel_joint: type continuous, parent base_link, child right_wheel_link, origin xyz=-0.1 -0.1 -0.015 rpy=0.0 0.0 0.0, axis 0.0 1.0 0.0

Commit message: tested

File: diffdrive_description/urdf/diffdrive.urdf (robot description, URDF)
Before this commit: robot DiffDrive, 2 links, 4 joints
Joints:
- removed joint front_joint
- added joint front_wheel_joint: type fixed, parent base_link, child front_wheel_link, origin xyz=0.1 0.0 -0.015 rpy=0.0 0.0 0.0

Commit message: add laser scan

File: diffdrive_description/urdf/diffdrive.urdf (robot description, URDF)
Before this commit: robot DiffDrive, 2 links, 4 joints
Links:
- added link front_wheel_link; visual sphere radius=0.03
